Commit message: UPDATE: URDF update

File: src/aero_hand_lite_description/urdf/aero_hand_lite_right.urdf (robot description, URDF)
Before this commit: robot aero_hand_lite_right, 22 links, 21 joints
Links:
- removed link  right_ring_middle_link
- removed link base_link
- removed link right_middle_link
- added link right_base_link, mass 0.303576106034272; collision mesh filename=package://aero_hand_lite_description/meshes/right_base_link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; visual mesh filename=package://aero_hand_lite_description/meshes/right_base_link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
- added link right_middle_middle_link, mass 0.00276150069139886; collision mesh filename=package://aero_hand_lite_description/meshes/right_middle_mi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; visual mesh filename=package://aero_hand_lite_description/meshes/right_middle_mi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
- added link right_ring_middle_link, mass 0.00276150640462905; collision mesh filename=package://aero_hand_lite_description/meshes/right_ring_midd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; visual mesh filename=package://aero_hand_lite_description/meshes/right_ring_midd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
Joints:
- joint right_index_mcp_flex: parent base_link -> right_base_link
- joint right_middle_dip: parent right_middle_link -> right_middle_middle_link
- joint right_middle_mcp_flex: parent base_link -> right_base_link
- joint right_middle_pip: child right_middle_link -> right_middle_middle_link
- joint right_pinky_mcp_flex: parent base_link -> right_base_link
- joint right_ring_dip: parent  right_ring_middle_link -> right_ring_middle_link
- joint right_ring_mcp_flex: parent base_link -> right_base_link
- joint right_ring_pip: child  right_ring_middle_link -> right_ring_middle_link
- joint right_thumb_cmc_abd: limit lower=-0.92502 upper=0.8203 effort=0 velocity=0 -> lower=0 upper=1.7453 effort=0 velocity=0; origin xyz=0.028112 -0.0145 0.025363 rpy=-1.3549 0.27644 -2.4646 -> xyz=0.028112 -0.0145 0.025363 rpy=-1.2217 -0.0 -1.57; parent base_link -> right_base_link
